File: MiniFeedMaster.sch (KiCad schematic (older format))
At the start: 33 parts, among them J1 SWD, J9 EXT, SW1 Button, SW2 Reset, U1 STM32F105Rx, Y1 25MHz ±10ppm 20pF 40Ω

Commit message: Added IO Protection Switched Fault Signal to +3.3V Added Voltage sensing Added correct UART pins to EXT header
Parts:
- added C50, C51: 100n, Capacitor_SMD:C_0603_1608Metric, symbol Device:C
- added R17, R31: 150k, Resistor_SMD:R_0603_1608Metric, symbol Device:R
- added R30, R32: 10k, Resistor_SMD:R_0603_1608Metric, symbol Device:R
Connections:
- net EXT_RX: now also U1.54 (PD2); no longer U1.33 (PB12)
- net EXT_TX: now also U1.53 (PC12); no longer U1.34 (PB13)
- net GND: now also U1.8 (PC0), C50.2, C51.2, R30.2, R32.2
- net at U1.10 (PC2): now also C51.1, R31.2, R32.1
- net at U1.16 (PA2): now also C50.1, R17.2, R30.1
- net FD_FAULT: no longer names the net of U1.59 (PB7)
- new net +12V: R17.1
- new net +24V: R31.1
- no-connect marks 26 -> 22

Commit message: Added LEDs to indicate power on the 12V and 3.3V rails Added Fiducials Moved references for SW1 and R2 Added 3D Model
Connections:
- no-connect marks 22 -> 24
Changed lines of the file:
@@
 Wire Wire Line
 	2100 3300 1300 3300
+NoConn ~ 4700 4300
+NoConn ~ 4700 4400
 $EndSCHEMATC
