File: can.sch (KiCad schematic (older format))
At the start: 18 parts, among them J2 CAN, U2 TPS76350, U3 SN6505B, U4 ISO1044

Commit message: Added LEDs to indicate power on the 12V and 3.3V rails Added Fiducials Moved references for SW1 and R2 Added 3D Model
Parts:
- C15, C16, C17, C18, C19, C20, C21, D2, D3, D4, J2, R7, R8, TR1, U2, U3, U4: Config (none) -> +can,-nocan
- FL1: Config (none) -> +can,-nocan; DNP (none) -> DNP
Changed lines of the file:
@@
 F 3 "https://www.ti.com/lit/ds/symlink/iso1044.pdf" H 3800 3100 50  0001 C CNN
 F 4 "ISO1044BD" H 3800 3100 50  0001 C CNN "manf#"
+F 5 "+can,-nocan" H 3800 3100 50  0001 C CNN "Config"
 	1    3800 3100
 	1    0    0    -1
@@
 F 4 "SN6505BDBVR" H 3100 1900 50  0001 C CNN "manf#"
 F 5 "C74518" H 3100 1900 50  0001 C CNN "lcsc#"
+F 6 "+can,-nocan" H 3100 1900 50  0001 C CNN "Config"
 	1    3100 1900
 	1    0    0    -1
@@
 F 4 "C194609" H 5900 1800 50  0001 C CNN "lcsc#"
 F 5 "TPS76350DBVR" H 5900 1800 50  0001 C CNN "manf#"
+F 6 "+can,-nocan" H 5900 1800 50  0001 C CNN "Config"
 	1    5900 1800
 	1    0    0    -1
@@
 F 3 "" H 3800 1900 50  0001 C CNN
 F 4 "760390015" H 3800 1900 50  0001 C CNN "manf#"
+F 5 "+can,-nocan" H 3800 1900 50  0001 C CNN "Config"
 	1    3800 1900
 	1    0    0    1
@@
 F 4 "C23848" H 4250 1700 50  0001 C CNN "lcsc#"
 F 5 "MBR0520LT1G" H 4250 1700 50  0001 C CNN "manf#"
+F 6 "+can,-nocan" H 4250 1700 50  0001 C CNN "Config"
 	1    4250 1700
 	-1   0    0    1
@@
 F 4 "C23848" H 4250 2100 50  0001 C CNN "lcsc#"
 F 5 "MBR0520LT1G" H 4250 2100 50  0001 C CNN "manf#"
+F 6 "+can,-nocan" H 4250 2100 50  0001 C CNN "Config"
 	1    4250 2100
 	-1   0    0    1
@@
 F 4 "C14860" H 4800 1950 50  0001 C CNN "lcsc#"
 F 5 "CL31B106KAHNNNE" H 4800 1950 50  0001 C CNN "manf#"
+F 6 "+can,-nocan" H 4800 1950 50  0001 C CNN "Config"
 	1    4800 1950
 	1    0    0    -1
@@
 F 4 "C1591" H 5200 1950 50  0001 C CNN "lcsc#"
 F 5 "CL10B104KB8NNNC" H 5200 1950 50  0001 C CNN "manf#"
+F 6 "+can,-nocan" H 5200 1950 50  0001 C CNN "Config"
 	1    5200 1950
 	1    0    0    -1
@@
 F 4 "C14860" H 6300 1950 50  0001 C CNN "lcsc#"
 F 5 "CL31B106KAHNNNE" H 6300 1950 50  0001 C CNN "manf#"
+F 6 "+can,-nocan" H 6300 1950 50  0001 C CNN "Config"
 	1    6300 1950
 	1    0    0    -1
@@
 F 4 "C1591" H 2000 1650 50  0001 C CNN "lcsc#"
 F 5 "CL10B104KB8NNNC" H 2000 1650 50  0001 C CNN "manf#"
+F 6 "+can,-nocan" H 2000 1650 50  0001 C CNN "Config"
 	1    2000 1650
 	1    0    0    -1
@@
 F 4 "ACT45B-510-2P-TL003" H 7000 3100 50  0001 C CNN "manf#"
 F 5 "C76584" H 7000 3100 50  0001 C CNN "lcsc#"
+F 6 "+can,-nocan" H 7000 3100 50  0001 C CNN "Config"
+F 7 "DNP" H 7000 3100 50  0001 C CNN "DNP"
 	1    7000 3100
 	1    0    0    -1
@@
 F 4 "C1591" H 4800 2550 50  0001 C CNN "lcsc#"
 F 5 "CL10B104KB8NNNC" H 4800 2550 50  0001 C CNN "manf#"
+F 6 "+can,-nocan" H 4800 2550 50  0001 C CNN "Config"
 	1    4800 2550
 	1    0    0    -1
@@
 F 4 "C163836" H 7050 3500 50  0001 C CNN "lcsc#"
 F 5 "WR06X0000FTL" H 7050 3500 50  0001 C CNN "manf#"
+F 6 "+can,-nocan" V 7050 3500 50  0001 C CNN "Config"
 	1    7050 3500
 	0    1    1    0
@@
 F 4 "C163836" H 7050 2700 50  0001 C CNN "lcsc#"
 F 5 "WR06X0000FTL" H 7050 2700 50  0001 C CNN "manf#"
+F 6 "+can,-nocan" V 7050 2700 50  0001 C CNN "Config"
 	1    7050 2700
 	0    1    1    0
@@
 F 4 "C246766" H 7600 3100 50  0001 C CNN "lcsc#"
 F 5 "ESDCAN24-2BLY" H 7600 3100 50  0001 C CNN "manf#"
+F 6 "+can,-nocan" V 7600 3100 50  0001 C CNN "Config"
 	1    7600 3100
 	0    -1   -1   0
@@
 F 4 "C475125" H 8800 2800 50  0001 C CNN "lcsc#"
 F 5 "KF141R-2.54-3P" H 8800 2800 50  0001 C CNN "manf#"
+F 6 "+can,-nocan" H 8800 2800 50  0001 C CNN "Config"
 	1    8800 2800
 	1    0    0    -1
@@
 F 4 "C14860" H 2000 3050 50  0001 C CNN "lcsc#"
 F 5 "CL31B106KAHNNNE" H 2000 3050 50  0001 C CNN "manf#"
+F 6 "+can,-nocan" H 2000 3050 50  0001 C CNN "Config"
 	1    2000 3050
 	1    0    0    -1
@@
 F 4 "C1591" H 2400 3050 50  0001 C CNN "lcsc#"
 F 5 "CL10B104KB8NNNC" H 2400 3050 50  0001 C CNN "manf#"
+F 6 "+can,-nocan" H 2400 3050 50  0001 C CNN "Config"
 	1    2400 3050
 	1    0    0    -1
